Commit message: Initial jazzy branch

File: amrROS2_ws/install/description/share/description/urdf/sensors/imu.urdf.xacro (robot description, xacro)
@@ -5,10 +5,15 @@
         <parent link="base_link"/>
         <child link="imu_frame"/>
-        <origin xyz="0.0245 -0.057 0.022" rpy="0 0 1.57"/>
+        <origin xyz="0.0245 -0.057 0.022" rpy="0 0 0"/>
       </joint>
-      <gazebo reference="imu_link">
+      <gazebo reference="imu_frame">
         <sensor name="imu_sensor" type="imu">
-          <ignition_frame_id>imu_link</ignition_frame_id>
+          <!-- <ignition_frame_id>imu_frame</ignition_frame_id>
           <plugin filename="ignition-gazebo-imu-system" name="ignition::gazebo::systems::Imu">
+          </plugin> -->
+          <pose relative_to='imu_frame'>0 0 0 0 0 0</pose>
+          <gz_frame_id>imu_frame</gz_frame_id>
+          <plugin filename="gz-sim-imu-system"
+                  name="gz::sim::systems::Imu">
           </plugin>
           <topic>imu</topic>

File: amrROS2_ws/src/description/urdf/controllers/diff_drive_controller.urdf.xacro (robot description, xacro)
@@ -2,5 +2,5 @@
 <robot xmlns:xacro="http://ros.org/wiki/xacro">
     <xacro:macro name="diff_drive_controller">
-        <ros2_control name="IgnitionSystem" type="system">
+        <!-- <ros2_control name="IgnitionSystem" type="system">
             <hardware>
             <plugin>ign_ros2_control/IgnitionSystem</plugin>
@@ -27,4 +27,36 @@
             <parameters>$(find gazebo)/config/controller.yaml</parameters>
             </plugin>
+        </gazebo> -->
+        <gazebo>
+            <plugin
+                filename="gz-sim-diff-drive-system"
+                name="gz::sim::systems::DiffDrive">
+                <left_joint>left_wheel_joint</left_joint>
+                <right_joint>right_wheel_joint</right_joint>
+                <wheel_separation>0.2254</wheel_separation>
+                <wheel_radius>0.0635</wheel_radius>
+                <max_linear_acceleration>1</max_linear_acceleration>
+                <min_linear_acceleration>-1</min_linear_acceleration>
+                <max_angular_acceleration>2</max_angular_acceleration>
+                <min_angular_acceleration>-2</min_angular_acceleration>
+                <max_linear_velocity>0.46</max_linear_velocity>
+                <min_linear_velocity>-0.46</min_linear_velocity>
+                <max_angular_velocity>1.9</max_angular_velocity>
+                <min_angular_velocity>-1.9</min_angular_velocity>
+                <topic>/cmd_vel</topic>
+                <odom_topic>/odom_raw</odom_topic>
+                <tf_topic>/tf</tf_topic>
+                <frame_id>odom</frame_id>
+                <child_frame_id>base_footprint</child_frame_id>
+                <odom_publish_frequency>40</odom_publish_frequency>
+            </plugin>
+            <plugin
+                filename="gz-sim-joint-state-publisher-system"
+                name="gz::sim::systems::JointStatePublisher">
+                <joint_name>left_wheel_joint</joint_name>
+                <joint_name>right_wheel_joint</joint_name>
+                <topic>/joint_states</topic>
+                <update_rate>40</update_rate>
+            </plugin>
         </gazebo>
     </xacro:macro>

File: amrROS2_ws/src/description/urdf/mech/wheel.urdf.xacro (robot description, xacro)
@@ -35,4 +35,11 @@
         </material>
       </visual>
+      <mu1>1000000000000000.0</mu1>
+      <mu2>1000000000000000.0</mu2>
+      <kp>1000000000000.0</kp>
+      <kd>10.0</kd>
+      <minDepth>0.001</minDepth>
+      <maxVel>0.1</maxVel>
+      <fdir1>1 0 0</fdir1>
     </gazebo>
     <joint name="${side}_wheel_joint" type="continuous">

File: amrROS2_ws/src/description/urdf/robot/robot.urdf.xacro (robot description, xacro)
@@ -10,5 +10,5 @@
   <xacro:include filename="$(find description)/urdf/sensors/camera.urdf.xacro" />
   <xacro:include filename="$(find description)/urdf/sensors/range_sensor.urdf.xacro" />
-  <!-- <xacro:diff_drive_controller/> -->
+  <xacro:diff_drive_controller/>
   <xacro:base
     length="${base_length}"

File: amrROS2_ws/src/description/urdf/sensors/imu.urdf.xacro (robot description, xacro)
@@ -5,11 +5,15 @@
         <parent link="base_link"/>
         <child link="imu_frame"/>
-        <!-- <origin xyz="0.0245 -0.057 0.022" rpy="0 0 1.57"/> -->
         <origin xyz="0.0245 -0.057 0.022" rpy="0 0 0"/>
       </joint>
-      <gazebo reference="imu_link">
+      <gazebo reference="imu_frame">
         <sensor name="imu_sensor" type="imu">
-          <ignition_frame_id>imu_link</ignition_frame_id>
+          <!-- <ignition_frame_id>imu_frame</ignition_frame_id>
           <plugin filename="ignition-gazebo-imu-system" name="ignition::gazebo::systems::Imu">
+          </plugin> -->
+          <pose relative_to='imu_frame'>0 0 0 0 0 0</pose>
+          <gz_frame_id>imu_frame</gz_frame_id>
+          <plugin filename="gz-sim-imu-system"
+                  name="gz::sim::systems::Imu">
           </plugin>
           <topic>imu</topic>

File: amrROS2_ws/src/description/urdf/sensors/laser.urdf.xacro (robot description, xacro)
@@ -41,30 +41,32 @@
       </joint>
       <gazebo reference="laser">
-        <sensor name="lidar" type="gpu_lidar">
-          <ignition_frame_id>laser</ignition_frame_id>
+        <sensor name='lidar' type='gpu_lidar'>
+          <pose relative_to='laser'>0 0 0 0 0 0</pose>
+          <gz_frame_id>laser</gz_frame_id>
           <topic>scan</topic>
-          <always_on>true</always_on>
+          <update_rate>40</update_rate>
+          <ray>
+              <scan>
+                  <horizontal>
+                      <samples>640</samples>
+                      <resolution>1</resolution>
+                      <min_angle>0.0</min_angle>
+                      <max_angle>6.28</max_angle>
+                  </horizontal>
+                  <vertical>
+                      <samples>1</samples>
+                      <resolution>0.01</resolution>
+                      <min_angle>0</min_angle>
+                      <max_angle>0</max_angle>
+                  </vertical>
+              </scan>
+              <range>
+                  <min>0.08</min>
+                  <max>10.0</max>
+                  <resolution>0.01</resolution>
+              </range>
+          </ray>
+          <always_on>1</always_on>
           <visualize>true</visualize>
-          <update_rate>30</update_rate>
-          <ray>
-            <scan>
-              <horizontal>
-                <samples>360</samples>
-                <resolution>1.000000</resolution>
-                <min_angle>0.000000</min_angle>
-                <max_angle>6.280000</max_angle>
-              </horizontal>
-            </scan>
-            <range>
-              <min>0.120000</min>
-              <max>10.0</max>
-              <resolution>0.015000</resolution>
-            </range>
-            <noise>
-              <type>gaussian</type>
-              <mean>0.0</mean>
-              <stddev>0.01</stddev>
-            </noise>
-          </ray>
         </sensor>
       </gazebo>

File: amrROS2_ws/src/description/urdf/sensors/range_sensor.urdf.xacro (robot description, xacro)
@@ -54,5 +54,5 @@
               </noise>
             </ray>
-            <plugin name="ultrasonic_sensor_1" filename="libgazebo_ros_ray_sensor.so">
+            <!-- <plugin name="ultrasonic_sensor_1" filename="libgazebo_ros_ray_sensor.so">
               <ros>
                 <remapping>~/out:=${pos}_range</remapping>
@@ -60,6 +60,6 @@
               <output_type>sensor_msgs/Range</output_type>
               <radiation_type>ultrasound</radiation_type>
-              <!-- <frame_name>${pos}_ranger_link</frame_name> -->
-            </plugin>
+              <frame_name>${pos}_ranger_link</frame_name>
+            </plugin> -->
           </sensor>
       </gazebo>
