Commit message: add gazebo

File: amrROS2_ws/src/description/urdf/controllers/diff_drive_controller.urdf.xacro (robot description, xacro)
@@ -2,5 +2,5 @@
 <robot xmlns:xacro="http://ros.org/wiki/xacro">
     <xacro:macro name="diff_drive_controller">
-        <ros2_control name="IgnitionSystem" type="system">
+        <!-- <ros2_control name="IgnitionSystem" type="system">
             <hardware>
             <plugin>ign_ros2_control/IgnitionSystem</plugin>
@@ -27,4 +27,36 @@
             <parameters>$(find gazebo)/config/controller.yaml</parameters>
             </plugin>
+        </gazebo> -->
+        <gazebo>
+            <plugin
+                filename="gz-sim-diff-drive-system"
+                name="gz::sim::systems::DiffDrive">
+                <left_joint>left_wheel_joint</left_joint>
+                <right_joint>right_wheel_joint</right_joint>
+                <wheel_separation>0.376</wheel_separation>
+                <wheel_radius>0.075</wheel_radius>
+                <max_linear_acceleration>1</max_linear_acceleration>
+                <min_linear_acceleration>-1</min_linear_acceleration>
+                <max_angular_acceleration>2</max_angular_acceleration>
+                <min_angular_acceleration>-2</min_angular_acceleration>
+                <max_linear_velocity>0.46</max_linear_velocity>
+                <min_linear_velocity>-0.46</min_linear_velocity>
+                <max_angular_velocity>1.9</max_angular_velocity>
+                <min_angular_velocity>-1.9</min_angular_velocity>
+                <topic>/cmd_vel</topic>
+                <odom_topic>/odom_raw</odom_topic>
+                <tf_topic>/tf</tf_topic>
+                <frame_id>odom</frame_id>
+                <child_frame_id>base_footprint</child_frame_id>
+                <odom_publish_frequency>40</odom_publish_frequency>
+            </plugin>
+            <plugin
+                filename="gz-sim-joint-state-publisher-system"
+                name="gz::sim::systems::JointStatePublisher">
+                <joint_name>left_wheel_joint</joint_name>
+                <joint_name>right_wheel_joint</joint_name>
+                <topic>/joint_states</topic>
+                <update_rate>40</update_rate>
+            </plugin>
         </gazebo>
     </xacro:macro>

File: amrROS2_ws/src/description/urdf/property/robot_property.urdf.xacro (robot description, xacro)
@@ -1,19 +1,19 @@
 <?xml version="1.0"?>
 <robot xmlns:xacro="http://ros.org/wiki/xacro">
-  <xacro:property name="base_length" value="0.345" />
-  <xacro:property name="base_width" value="0.2" />
-  <xacro:property name="base_height" value="0.14" />
-  <xacro:property name="base_mass" value="3" />
-  <xacro:property name="wheel_radius" value="0.0635" />
-  <xacro:property name="wheel_width" value="0.0254" />
-  <xacro:property name="wheel_pos_x" value="0.0725" />
-  <xacro:property name="wheel_pos_y" value="0.11" />
-  <xacro:property name="wheel_pos_z" value="-0.045" />
-  <xacro:property name="wheel_mass" value="2.5" />
+  <xacro:property name="base_length" value="0.48" />
+  <xacro:property name="base_width" value="0.42" />
+  <xacro:property name="base_height" value="0.24" />
+  <xacro:property name="base_mass" value="30" />
+  <xacro:property name="wheel_radius" value="0.075" />
+  <xacro:property name="wheel_width" value="0.04" />
+  <xacro:property name="wheel_pos_x" value="0.0" />
+  <xacro:property name="wheel_pos_y" value="0.168" />
+  <xacro:property name="wheel_pos_z" value="-0.115" />
+  <xacro:property name="wheel_mass" value="1.236" />
   <xacro:property name="wheel_torque" value="20" />
-  <xacro:property name="front_caster_wheel" value="false" />
-  <xacro:property name="rear_caster_wheel" value="false" />
-  <xacro:property name="left_caster_wheel" value="true" />
-  <xacro:property name="right_caster_wheel" value="true" />
+  <!-- <xacro:property name="front_caster_wheel" value="true" />
+  <xacro:property name="rear_caster_wheel" value="true" />
+  <xacro:property name="left_caster_wheel" value="false" />
+  <xacro:property name="right_caster_wheel" value="false" /> -->
   <!-- <xacro:property name="laser_pose">
     <origin xyz="0.12 0 0.33" rpy="0 0 0"/>

File: amrROS2_ws/src/description/urdf/robot/robot.urdf.xacro (robot description, xacro)
@@ -10,5 +10,5 @@
   <xacro:include filename="$(find description)/urdf/sensors/camera.urdf.xacro" />
   <xacro:include filename="$(find description)/urdf/sensors/range_sensor.urdf.xacro" />
-  <!-- <xacro:diff_drive_controller/> -->
+  <xacro:diff_drive_controller/>
   <xacro:base
     length="${base_length}"
@@ -39,5 +39,5 @@
   />
   <xacro:caster_wheel
-      side="right"
+      side="front"
       mass="0.01"
       base_length="${base_length}"
@@ -48,5 +48,5 @@
     />
     <xacro:caster_wheel
-      side="left"
+      side="rear"
       mass="0.01"
       base_length="${base_length}"
@@ -59,5 +59,5 @@
   <xacro:imu/>
   <xacro:laser/>
-  <xacro:range_sensor
+  <!-- <xacro:range_sensor
     pos="center"
     pos_x="0.1725"
@@ -82,5 +82,5 @@
     pitch="0"
     yaw="-0.6106"
-  />
+  /> -->
   <!-- <xacro:depth_sensor>
     <xacro:insert_block name="depth_sensor_pose" />

File: amrROS2_ws/src/description/urdf/sensors/camera.urdf.xacro (robot description, xacro)
@@ -1,5 +1,5 @@
 <robot xmlns:xacro="http://ros.org/wiki/xacro">
     <xacro:macro name="camera">
-      <link name="camera">
+      <link name="rgbd_frame">
         <visual>
           <origin xyz="0 0 0" rpy="0 0 0"/>
@@ -27,27 +27,68 @@
       <joint name="camera_to_base_link" type="fixed">
         <parent link="base_link"/>
-        <child link="camera" />
-        <origin xyz="0.1475 0.0 0.055" rpy="0 0 0"/>
+        <child link="rgbd_frame" />
+        <origin xyz="0.24 0.0 0.12" rpy="0 0 0"/>
       </joint>
-         <gazebo reference="camera">
-            <sensor name="robot_cam" type="camera">
-              <camera>
-                <horizontal_fov>1.047</horizontal_fov>
-                <image>
-                  <width>320</width>
-                  <height>240</height>
-                </image>
-                <clip>
-                  <near>0.1</near>
-                  <far>100</far>
-                </clip>
-              </camera>
-              <always_on>1</always_on>
-              <update_rate>30</update_rate>
-              <visualize>true</visualize>
-              <topic>robot_cam</topic>
-              <enable_metrics>true</enable_metrics>
-            </sensor>
-          </gazebo>
+      <!-- <gazebo reference="camera">
+        <sensor name="robot_cam" type="camera">
+          <camera>
+            <horizontal_fov>1.047</horizontal_fov>
+            <image>
+              <width>320</width>
+              <height>240</height>
+            </image>
+            <clip>
+              <near>0.1</near>
+              <far>100</far>
+            </clip>
+          </camera>
+          <always_on>1</always_on>
+          <update_rate>30</update_rate>
+          <visualize>true</visualize>
+          <topic>robot_cam</topic>
+          <enable_metrics>true</enable_metrics>
+        </sensor>
+      </gazebo> -->
+      <gazebo reference="rgbd_frame">
+      <sensor type="depth" name="rgbd_sensor">
+        <always_on>true</always_on>
+        <update_rate>30.0</update_rate>
+        <gz_frame_id>rgbd_frame</gz_frame_id>
+        <topic>robot_cam</topic>
+        <camera>
+          <horizontal_fov>${63.0*3.144159265/180.0}</horizontal_fov>
+          <image>
+            <format>B8G8R8</format>
+            <width>640</width>
+            <height>480</height>
+          </image>
+          <clip>z
+            <near>0.1</near>
+            <far>8.0</far>
+          </clip>
+          <distortion>
+            <k1>0.00000001</k1>
+            <k2>0.00000001</k2>
+            <k3>0.00000001</k3>
+            <p1>0.00000001</p1>
+            <p2>0.00000001</p2>
+          </distortion>
+        </camera>
+        <plugin name="rgbd_frame_controller" filename="libgazebo_ros_camera.so">
+          <camera_name>rgbd</camera_name>
+          <!-- <ros> -->
+            <!-- <namespace>${name}</namespace> -->
+            <!-- <remapping>rgbd/image_raw:=rgbd/rgb/image_raw</remapping>
+            <remapping>rgbd/camera_info:=rgbd/rgb/camera_info</remapping>
+            <remapping>rgbd/depth/image_raw:=rgbd/depth_registered/image_raw</remapping>
+            <remapping>rgbd/depth/camera_info:=rgbd/depth_registered/camera_info</remapping>
+            <remapping>rgbd/points:=rgbd/depth_registered/points</remapping> -->
+          <!-- </ros> -->
+          <frame_name>rgbd_frame</frame_name>
+          <min_depth>0.1</min_depth>
+          <max_depth>8.0</max_depth>
+        </plugin>
+      </sensor>
+    </gazebo>
     </xacro:macro>
 </robot>

File: amrROS2_ws/src/description/urdf/sensors/imu.urdf.xacro (robot description, xacro)
@@ -5,11 +5,12 @@
         <parent link="base_link"/>
         <child link="imu_frame"/>
-        <!-- <origin xyz="0.0245 -0.057 0.022" rpy="0 0 1.57"/> -->
         <origin xyz="0.0245 -0.057 0.022" rpy="0 0 0"/>
       </joint>
-      <gazebo reference="imu_link">
+      <gazebo reference="imu_frame">
         <sensor name="imu_sensor" type="imu">
-          <ignition_frame_id>imu_link</ignition_frame_id>
-          <plugin filename="ignition-gazebo-imu-system" name="ignition::gazebo::systems::Imu">
+          <pose relative_to='imu_frame'>0 0 0 0 0 0</pose>
+          <gz_frame_id>imu_frame</gz_frame_id>
+          <plugin filename="gz-sim-imu-system"
+                  name="gz::sim::systems::Imu">
           </plugin>
           <topic>imu</topic>

File: amrROS2_ws/src/description/urdf/sensors/laser.urdf.xacro (robot description, xacro)
@@ -5,5 +5,5 @@
           <origin xyz="0 0 0" rpy="0 0 0"/>
           <geometry>
-            <cylinder length="0.0182" radius="0.0255"/>
+            <cylinder length="0.05" radius="0.0375"/>
           </geometry>
           <material name="green">
@@ -14,5 +14,5 @@
           <origin xyz="0 0 0" rpy="0 0 0"/>
           <geometry>
-            <cylinder length="0.0182" radius="0.0255"/>
+            <cylinder length="0.05" radius="0.0375"/>
           </geometry>
         </collision>
@@ -38,33 +38,35 @@
         <parent link="base_link"/>
         <child link="laser"/>
-        <origin xyz="0.0925 0 0.0791" rpy="0 0 3.14"/>
+        <origin xyz="0.0 0 0.21" rpy="0 0 3.144159265"/>
       </joint>
       <gazebo reference="laser">
-        <sensor name="lidar" type="gpu_lidar">
-          <ignition_frame_id>laser</ignition_frame_id>
+        <sensor name='lidar' type='gpu_lidar'>
+          <pose relative_to='laser'>0 0 0 0 0 0</pose>
+          <gz_frame_id>laser</gz_frame_id>
           <topic>scan</topic>
-          <always_on>true</always_on>
+          <update_rate>40</update_rate>
+          <ray>
+              <scan>
+                  <horizontal>
+                      <samples>640</samples>
+                      <resolution>1</resolution>
+                      <min_angle>0.0</min_angle>
+                      <max_angle>6.28</max_angle>
+                  </horizontal>
+                  <vertical>
+                      <samples>1</samples>
+                      <resolution>0.01</resolution>
+                      <min_angle>0</min_angle>
+                      <max_angle>0</max_angle>
+                  </vertical>
+              </scan>
+              <range>
+                  <min>0.08</min>
+                  <max>10.0</max>
+                  <resolution>0.01</resolution>
+              </range>
+          </ray>
+          <always_on>1</always_on>
           <visualize>true</visualize>
-          <update_rate>30</update_rate>
-          <ray>
-            <scan>
-              <horizontal>
-                <samples>360</samples>
-                <resolution>1.000000</resolution>
-                <min_angle>0.000000</min_angle>
-                <max_angle>6.280000</max_angle>
-              </horizontal>
-            </scan>
-            <range>
-              <min>0.120000</min>
-              <max>10.0</max>
-              <resolution>0.015000</resolution>
-            </range>
-            <noise>
-              <type>gaussian</type>
-              <mean>0.0</mean>
-              <stddev>0.01</stddev>
-            </noise>
-          </ray>
         </sensor>
       </gazebo>

Commit message: first commit in realhardware

File: amrROS2_ws/src/description/urdf/controllers/diff_drive_controller.urdf.xacro (robot description, xacro)
@@ -2,30 +2,4 @@
 <robot xmlns:xacro="http://ros.org/wiki/xacro">
     <xacro:macro name="diff_drive_controller">
-        <!-- <ros2_control name="IgnitionSystem" type="system">
-            <hardware>
-            <plugin>ign_ros2_control/IgnitionSystem</plugin>
-            </hardware>
-            <joint name="left_wheel_joint">
-            <command_interface name="velocity">
-                <param name="min">-1</param>
-                <param name="max">1</param>
-            </command_interface>
-            <state_interface name="position"/>
-            <state_interface name="velocity"/>
-            </joint>
-            <joint name="right_wheel_joint">
-            <command_interface name="velocity">
-                <param name="min">-1</param>
-                <param name="max">1</param>
-            </command_interface>
-            <state_interface name="position"/>
-            <state_interface name="velocity"/>
-            </joint>
-        </ros2_control>
-        <gazebo>
-            <plugin filename="ign_ros2_control-system" name="ign_ros2_control::IgnitionROS2ControlPlugin">
-            <parameters>$(find gazebo)/config/controller.yaml</parameters>
-            </plugin>
-        </gazebo> -->
         <gazebo>
             <plugin

File: amrROS2_ws/src/description/urdf/robot/robot.urdf.xacro (robot description, xacro)
@@ -10,5 +10,5 @@
   <xacro:include filename="$(find description)/urdf/sensors/camera.urdf.xacro" />
   <xacro:include filename="$(find description)/urdf/sensors/range_sensor.urdf.xacro" />
-  <xacro:diff_drive_controller/>
+  <!-- <xacro:diff_drive_controller/> -->
   <xacro:base
     length="${base_length}"

File: amrROS2_ws/src/description/urdf/sensors/laser.urdf.xacro (robot description, xacro)
@@ -38,5 +38,5 @@
         <parent link="base_link"/>
         <child link="laser"/>
-        <origin xyz="0.0 0 0.21" rpy="0 0 3.144159265"/>
+        <origin xyz="0.0 0 0.055" rpy="0 0 3.144159265"/>
       </joint>
       <gazebo reference="laser">

File: amrROS2_ws/src/description/urdf/sensors/range_sensor.urdf.xacro (robot description, xacro)
@@ -60,5 +60,4 @@
               <output_type>sensor_msgs/Range</output_type>
               <radiation_type>ultrasound</radiation_type>
-              <!-- <frame_name>${pos}_ranger_link</frame_name> -->
             </plugin>
           </sensor>
