Commit message: update

File: amrROS2_ws/src/description/urdf/sensors/imu.urdf.xacro (robot description, xacro)
@@ -5,5 +5,6 @@
         <parent link="base_link"/>
         <child link="imu_frame"/>
-        <origin xyz="0.0245 -0.057 0.022" rpy="0 0 1.57"/>
+        <!-- <origin xyz="0.0245 -0.057 0.022" rpy="0 0 1.57"/> -->
+        <origin xyz="0.0245 -0.057 0.022" rpy="0 0 0"/>
       </joint>
       <gazebo reference="imu_link">

Commit message: creat thai-easy branch

File: amrROS2_ws/src/description/urdf/sensors/imu.urdf.xacro (robot description, xacro)
@@ -5,5 +5,5 @@
         <parent link="base_link"/>
         <child link="imu_frame"/>
-        <origin xyz="0.0245 -0.057 0.022" rpy="0 0 0"/>
+        <origin xyz="0.05 0 0.022" rpy="0 0 0"/>
       </joint>
       <gazebo reference="imu_frame">
